Commit message: Added a laser scanner sensor

File: neato_description/urdf/neato.urdf.xacro (robot description, xacro)
@@ -27,13 +27,13 @@
       <collision>
         <geometry>
-          <cylinder length="0.08" radius="0.15"/>
-        </geometry>
-        <origin xyz="-0.01 0 0.04" rpy="0 0 0"/>
-      </collision>
-      <collision>
-        <geometry>
-          <box size="0.16 0.3 0.08"/>
-        </geometry>
-        <origin xyz="0.08 0 0.04" rpy="0 0 0"/>
+          <cylinder length="0.06" radius="0.15"/>
+        </geometry>
+        <origin xyz="-0.01 0 0.03" rpy="0 0 0"/>
+      </collision>
+      <collision>
+        <geometry>
+          <box size="0.16 0.3 0.06"/>
+        </geometry>
+        <origin xyz="0.08 0 0.03" rpy="0 0 0"/>
       </collision>
       <inertial>
@@ -196,5 +196,5 @@
     </link>
     <joint name="cliff_sensor_right_joint" type="fixed">
-      <origin xyz="0.11 -${0.29/2} 0" rpy="0 0 0" />
+      <origin xyz="0.11 -${0.29/2} 0" rpy="0 ${M_PI/2} 0" />
       <parent link="base_link"/>
       <child link="cliff_sensor_right_link" />
@@ -210,5 +210,5 @@
     </link>
     <joint name="cliff_sensor_left_joint" type="fixed">
-      <origin xyz="0.11 ${0.29/2} 0" rpy="0 0 0" />
+      <origin xyz="0.11 ${0.29/2} 0" rpy="0 ${M_PI/2} 0" />
       <parent link="base_link"/>
       <child link="cliff_sensor_left_link" />
@@ -223,4 +223,18 @@
       </inertial>
     </link>
+    <joint name="laser_joint" type="fixed">
+      <origin xyz="-0.084 0 0.066" rpy="0 0 0" />
+      <parent link="base_link"/>
+      <child link="laser_link" />
+    </joint>
+    <link name="laser_link">
+      <inertial>
+        <mass value="0.0001" />
+        <origin xyz="0 0 0" />
+        <inertia ixx="0.0001" ixy="0.0" ixz="0.0"
+                 iyy="0.0001" iyz="0.0"
+                 izz="0.0001" />
+      </inertial>
+    </link>
     <neato_sim/>
   </xacro:macro>

File: neato_description/urdf/neato_gazebo.urdf.xacro (robot description, xacro)
@@ -2,129 +2,139 @@
 <robot name="neato_sim" xmlns:xacro="http://ros.org/wiki/xacro">
   <xacro:macro name="neato_sim">
-          <gazebo reference="base_link">
-            <material>Gazebo/DarkGrey</material>
-          </gazebo>
-	  <gazebo reference="wheel_left_link">
-	    <mu1>1.0</mu1>
-	    <mu2>1.0</mu2>
-	    <kp>1000000.0</kp>
-	    <kd>100.0</kd>
-	    <minDepth>0.001</minDepth>
-	    <maxVel>1.0</maxVel>
-	  </gazebo>
-	  <gazebo reference="wheel_right_link">
-	    <mu1>1.0</mu1>
-	    <mu2>1.0</mu2>
-	    <kp>1000000.0</kp>
-	    <kd>100.0</kd>
-	    <minDepth>0.001</minDepth>
-	    <maxVel>1.0</maxVel>
-	  </gazebo>
-	  <gazebo reference="caster_front_right_link">
-	    <mu1>0.0</mu1>
-	    <mu2>0.0</mu2>
-	    <kp>1000000.0</kp>
-	    <kd>100.0</kd>
-	    <minDepth>0.001</minDepth>
-	    <maxVel>1.0</maxVel>
-	  </gazebo>
-	  <gazebo reference="caster_front_left_link">
-	    <mu1>0.0</mu1>
-	    <mu2>0.0</mu2>
-	    <kp>1000000.0</kp>
-	    <kd>100.0</kd>
-	    <minDepth>0.001</minDepth>
-	    <maxVel>1.0</maxVel>
-	  </gazebo>
-	  <gazebo reference="caster_back_right_link">
-	    <mu1>0.0</mu1>
-	    <mu2>0.0</mu2>
-	    <kp>1000000.0</kp>
-	    <kd>100.0</kd>
-	    <minDepth>0.001</minDepth>
-	    <maxVel>1.0</maxVel>
-	  </gazebo>
-	  <gazebo reference="caster_back_left_link">
-	    <mu1>0.0</mu1>
-	    <mu2>0.0</mu2>
-	    <kp>1000000.0</kp>
-	    <kd>100.0</kd>
-	    <minDepth>0.001</minDepth>
-	    <maxVel>1.0</maxVel>
-	  </gazebo>
-	  <gazebo reference="base_link">
-	    <mu1>0.3</mu1>
-	    <mu2>0.3</mu2>
-	    <sensor type="contact" name="bumpers">
-	      <always_on>1</always_on>
-	      <update_rate>50.0</update_rate>
-	      <visualize>true</visualize>
-	      <contact>
-	        <collision>base_footprint_collision_base_link</collision>
-	      </contact>
-	    </sensor>
-	  </gazebo>
-	  <gazebo reference="cliff_sensor_left_link">
-	    <sensor type="ray" name="cliff_sensor_left">
-	      <always_on>true</always_on>
-	      <update_rate>50</update_rate>
-	      <visualize>true</visualize>
-	      <ray>
-	        <scan>
-	          <horizontal>
-	            <samples>50</samples>
-	            <resolution>1.0</resolution>
-	            <min_angle>-0.0436</min_angle>  <!-- -2.5 degree -->
-	            <max_angle>0.0436</max_angle> <!-- 2.5 degree -->
-	          </horizontal>
-<!--            Can't use vertical rays until this bug is resolved: -->
-<!--            https://bitbucket.org/osrf/gazebo/issue/509/vertical-sensor-doesnt-works -->
-<!-- 	          <vertical> -->
-<!-- 	            <samples>50</samples> -->
-<!-- 	            <resolution>1.0</resolution> -->
-<!-- 	            <min_angle>-0.0436</min_angle>  -2.5 degree -->
-<!-- 	            <max_angle>0.0436</max_angle> 2.5 degree -->
-<!-- 	          </vertical> -->
-	        </scan>
-	        <range>
-	          <min>0.01</min>
-	          <max>0.15</max>
-	          <resolution>1.0</resolution>
-	        </range>
-	      </ray>
-	    </sensor>
-	  </gazebo>
-	  <gazebo reference="cliff_sensor_right_link">
-	    <sensor type="ray" name="cliff_sensor_right">
-	      <always_on>true</always_on>
-	      <update_rate>50</update_rate>
-	      <visualize>true</visualize>
-	      <ray>
-	        <scan>
-	          <horizontal>
-	            <samples>50</samples>
-	            <resolution>1.0</resolution>
-	            <min_angle>-0.0436</min_angle>  <!-- -2.5 degree -->
-	            <max_angle>0.0436</max_angle> <!-- 2.5 degree -->
-	          </horizontal>
-<!--            Can't use vertical rays until this bug is resolved: -->
-<!--            https://bitbucket.org/osrf/gazebo/issue/509/vertical-sensor-doesnt-works -->
-<!-- 	          <vertical> -->
-<!-- 	            <samples>50</samples> -->
-<!-- 	            <resolution>1.0</resolution> -->
-<!-- 	            <min_angle>-0.0436</min_angle>  -2.5 degree -->
-<!-- 	            <max_angle>0.0436</max_angle> 2.5 degree -->
-<!-- 	          </vertical> -->
-	        </scan>
-	        <range>
-	          <min>0.01</min>
-	          <max>0.15</max>
-	          <resolution>1.0</resolution>
-	        </range>
-	      </ray>
-	    </sensor>
-	  </gazebo>
-	  <gazebo reference="gyro_link">
-	   <sensor type="imu" name="imu">
+    <gazebo reference="base_link">
+      <material>Gazebo/DarkGrey</material>
+    </gazebo>
+    <gazebo reference="wheel_left_link">
+      <mu1>1.0</mu1>
+      <mu2>1.0</mu2>
+      <kp>1000000.0</kp>
+      <kd>100.0</kd>
+      <minDepth>0.001</minDepth>
+      <maxVel>1.0</maxVel>
+    </gazebo>
+    <gazebo reference="wheel_right_link">
+      <mu1>1.0</mu1>
+      <mu2>1.0</mu2>
+      <kp>1000000.0</kp>
+      <kd>100.0</kd>
+      <minDepth>0.001</minDepth>
+      <maxVel>1.0</maxVel>
+    </gazebo>
+    <gazebo reference="caster_front_right_link">
+      <mu1>0.0</mu1>
+      <mu2>0.0</mu2>
+      <kp>1000000.0</kp>
+      <kd>100.0</kd>
+      <minDepth>0.001</minDepth>
+      <maxVel>1.0</maxVel>
+    </gazebo>
+    <gazebo reference="caster_front_left_link">
+      <mu1>0.0</mu1>
+      <mu2>0.0</mu2>
+      <kp>1000000.0</kp>
+      <kd>100.0</kd>
+      <minDepth>0.001</minDepth>
+      <maxVel>1.0</maxVel>
+    </gazebo>
+    <gazebo reference="caster_back_right_link">
+      <mu1>0.0</mu1>
+      <mu2>0.0</mu2>
+      <kp>1000000.0</kp>
+      <kd>100.0</kd>
+      <minDepth>0.001</minDepth>
+      <maxVel>1.0</maxVel>
+    </gazebo>
+    <gazebo reference="caster_back_left_link">
+      <mu1>0.0</mu1>
+      <mu2>0.0</mu2>
+      <kp>1000000.0</kp>
+      <kd>100.0</kd>
+      <minDepth>0.001</minDepth>
+      <maxVel>1.0</maxVel>
+    </gazebo>
+    <gazebo reference="base_link">
+      <mu1>0.3</mu1>
+      <mu2>0.3</mu2>
+      <sensor type="contact" name="bumpers">
+        <always_on>1</always_on>
+        <update_rate>50.0</update_rate>
+        <visualize>true</visualize>
+        <contact>
+          <collision>base_footprint_collision_base_link</collision>
+        </contact>
+      </sensor>
+    </gazebo>
+    <gazebo reference="cliff_sensor_left_link">
+      <sensor type="ray" name="cliff_sensor_left">
+        <always_on>true</always_on>
+        <update_rate>50</update_rate>
+        <visualize>true</visualize>
+        <ray>
+          <scan>
+            <horizontal>
+              <samples>50</samples>
+              <resolution>1.0</resolution>
+              <min_angle>-0.0436</min_angle>
+              <max_angle>0.0436</max_angle>
+            </horizontal>
+          </scan>
+          <range>
+            <min>0.01</min>
+            <max>0.15</max>
+            <resolution>1.0</resolution>
+          </range>
+        </ray>
+      </sensor>
+    </gazebo>
+    <gazebo reference="cliff_sensor_right_link">
+      <sensor type="ray" name="cliff_sensor_right">
+        <always_on>true</always_on>
+        <update_rate>50</update_rate>
+        <visualize>true</visualize>
+        <ray>
+          <scan>
+            <horizontal>
+              <samples>50</samples>
+              <resolution>1.0</resolution>
+              <min_angle>-0.0436</min_angle>
+              <max_angle>0.0436</max_angle>
+            </horizontal>
+          </scan>
+          <range>
+            <min>0.01</min>
+            <max>0.15</max>
+            <resolution>1.0</resolution>
+          </range>
+        </ray>
+      </sensor>
+    </gazebo>
+    <gazebo reference="laser_link">
+      <sensor type="gpu_ray" name="laser">
+        <always_on>true</always_on>
+        <update_rate>50</update_rate>
+        <visualize>true</visualize>
+        <ray>
+          <scan>
+            <horizontal>
+              <samples>360</samples>
+              <resolution>1</resolution>
+              <min_angle>${-M_PI}</min_angle>
+              <max_angle>${M_PI}</max_angle>
+            </horizontal>
+          </scan>
+          <range>
+            <min>0.1</min>
+            <max>5</max>
+            <resolution>1</resolution>
+          </range>
+        </ray>
+        <plugin name="gazebo_ros_laser_controller" filename="libgazebo_ros_gpu_laser.so">
+          <topicName>/neato/laser/scan</topicName>
+          <frameName>laser_link</frameName>
+        </plugin>
+      </sensor>
+    </gazebo>
+    <gazebo reference="gyro_link">
+      <sensor type="imu" name="imu">
         <always_on>true</always_on>
         <update_rate>50</update_rate>
@@ -133,36 +143,36 @@
           <noise>
             <type>gaussian</type>
-	          <rate>
-	            <mean>0.0</mean>
-	            <stddev>${0.0014*0.0014}</stddev> <!-- 0.25 x 0.25 (deg/s) -->
-	            <bias_mean>0.0</bias_mean>
-	            <bias_stddev>0.0</bias_stddev>
-	          </rate>
-		        <accel> <!-- not used in the plugin and real robot, hence using tutorial values -->
-			        <mean>0.0</mean>
-			        <stddev>1.7e-2</stddev>
-			        <bias_mean>0.1</bias_mean>
-			        <bias_stddev>0.001</bias_stddev>
-		        </accel>
+            <rate>
+              <mean>0.0</mean>
+              <stddev>${0.0014*0.0014}</stddev>
+              <bias_mean>0.0</bias_mean>
+              <bias_stddev>0.0</bias_stddev>
+            </rate>
+            <accel>
+              <mean>0.0</mean>
+              <stddev>1.7e-2</stddev>
+              <bias_mean>0.1</bias_mean>
+              <bias_stddev>0.001</bias_stddev>
+            </accel>
           </noise>
-	      </imu>
+        </imu>
       </sensor>
-	  </gazebo>
-	  <gazebo>
-	    <plugin name="neato_controller" filename="libgazebo_ros_neato.so">
-	      <publish_tf>1</publish_tf>
-	      <left_wheel_joint_name>wheel_left_joint</left_wheel_joint_name>
-	      <right_wheel_joint_name>wheel_right_joint</right_wheel_joint_name>
-	      <wheel_separation>.230</wheel_separation>
-	      <wheel_diameter>0.070</wheel_diameter>
-	      <torque>1.0</torque>
-	      <velocity_command_timeout>0.6</velocity_command_timeout>
-	      <cliff_sensor_left_name>cliff_sensor_left</cliff_sensor_left_name>
-	      <cliff_sensor_right_name>cliff_sensor_right</cliff_sensor_right_name>
-	      <cliff_detection_threshold>0.04</cliff_detection_threshold>
-	      <bumper_name>bumpers</bumper_name>
-              <imu_name>imu</imu_name>
-	    </plugin>
-	  </gazebo>
+    </gazebo>
+    <gazebo>
+      <plugin name="neato_controller" filename="libgazebo_ros_neato.so">
+        <publish_tf>1</publish_tf>
+        <left_wheel_joint_name>wheel_left_joint</left_wheel_joint_name>
+        <right_wheel_joint_name>wheel_right_joint</right_wheel_joint_name>
+        <wheel_separation>.230</wheel_separation>
+        <wheel_diameter>0.070</wheel_diameter>
+        <torque>1.0</torque>
+        <velocity_command_timeout>0.6</velocity_command_timeout>
+        <cliff_sensor_left_name>cliff_sensor_left</cliff_sensor_left_name>
+        <cliff_sensor_right_name>cliff_sensor_right</cliff_sensor_right_name>
+        <cliff_detection_threshold>0.04</cliff_detection_threshold>
+        <bumper_name>bumpers</bumper_name>
+        <imu_name>imu</imu_name>
+      </plugin>
+    </gazebo>
   </xacro:macro>
 </robot>

Commit message: Made the Neato robot compatible with the Kobuki Keyop

File: neato_description/urdf/neato.urdf.xacro (robot description, xacro)
@@ -48,5 +48,5 @@
       <parent link="base_link"/>
       <child link="wheel_left_link"/>
-      <origin xyz="0.00 ${0.235/2} 0.0250" rpy="${M_PI/2} 0 0"/>
+      <origin xyz="0.00 ${0.235/2} 0.0250" rpy="${M_PI/2} 0 ${M_PI}"/>
       <axis xyz="0 0 1"/>
     </joint>
@@ -75,5 +75,5 @@
       <parent link="base_link"/>
       <child link="wheel_right_link"/>
-      <origin xyz="0.00 -${0.235/2} 0.0250" rpy="${M_PI/2} 0 0"/>
+      <origin xyz="0.00 -${0.235/2} 0.0250" rpy="${M_PI/2} 0 ${M_PI}"/>
       <axis xyz="0 0 1"/>
     </joint>

File: neato_description/urdf/neato_gazebo.urdf.xacro (robot description, xacro)
@@ -164,5 +164,5 @@
         <left_wheel_joint_name>wheel_left_joint</left_wheel_joint_name>
         <right_wheel_joint_name>wheel_right_joint</right_wheel_joint_name>
-        <wheel_separation>.230</wheel_separation>
+        <wheel_separation>0.235</wheel_separation>
         <wheel_diameter>0.070</wheel_diameter>
         <torque>1.0</torque>

Commit message: Changed to standard Gazebo-ROS plugins for sensors and actuators in package neato_gazebo. This deprecates packages neato_gazebo_plugins.

File: neato_description/urdf/neato.urdf.xacro (robot description, xacro)
@@ -180,11 +180,11 @@
     </link>
     <!-- neato's sensors -->
-    <joint name="gyro_joint" type="fixed">
+    <joint name="imu_joint" type="fixed">
       <axis xyz="0 1 0"/>
       <origin xyz="0 0 0" rpy="0 0 0"/>
       <parent link="base_link"/>
-      <child link="gyro_link"/>
-    </joint>
-    <link name="gyro_link">
+      <child link="imu_link"/>
+    </joint>
+    <link name="imu_link">
       <inertial>
         <mass value="0.001"/>

File: neato_description/urdf/neato_gazebo.urdf.xacro (robot description, xacro)
@@ -63,8 +63,12 @@
           <collision>base_footprint_collision_base_link</collision>
         </contact>
+        <plugin name="gazebo_ros_bumper_controller" filename="libgazebo_ros_bumper.so">
+          <bumperTopicName>/neato/bumper</bumperTopicName>
+          <frameName>world</frameName>
+        </plugin>
       </sensor>
     </gazebo>
     <gazebo reference="cliff_sensor_left_link">
-      <sensor type="ray" name="cliff_sensor_left">
+      <sensor type="gpu_ray" name="cliff_sensor_left">
         <always_on>true</always_on>
         <update_rate>50</update_rate>
@@ -85,8 +89,12 @@
           </range>
         </ray>
+        <plugin name="gazebo_ros_laser_controller" filename="libgazebo_ros_gpu_laser.so">
+          <topicName>/neato/cliff_left</topicName>
+          <frameName>cliff_sensor_left_link</frameName>
+        </plugin>
       </sensor>
     </gazebo>
     <gazebo reference="cliff_sensor_right_link">
-      <sensor type="ray" name="cliff_sensor_right">
+      <sensor type="gpu_ray" name="cliff_sensor_right">
         <always_on>true</always_on>
         <update_rate>50</update_rate>
@@ -107,4 +115,8 @@
           </range>
         </ray>
+        <plugin name="gazebo_ros_laser_controller" filename="libgazebo_ros_gpu_laser.so">
+          <topicName>/neato/cliff_right</topicName>
+          <frameName>cliff_sensor_right_link</frameName>
+        </plugin>
       </sensor>
     </gazebo>
@@ -130,10 +142,10 @@
         </ray>
         <plugin name="gazebo_ros_laser_controller" filename="libgazebo_ros_gpu_laser.so">
-          <topicName>/neato/laser/scan</topicName>
+          <topicName>/neato/laser</topicName>
           <frameName>laser_link</frameName>
         </plugin>
       </sensor>
     </gazebo>
-    <gazebo reference="gyro_link">
+    <gazebo reference="imu_link">
       <sensor type="imu" name="imu">
         <always_on>true</always_on>
@@ -160,19 +172,24 @@
     </gazebo>
     <gazebo>
-      <plugin name="neato_controller" filename="libgazebo_ros_neato.so">
-        <publish_tf>1</publish_tf>
-        <left_wheel_joint_name>wheel_left_joint</left_wheel_joint_name>
-        <right_wheel_joint_name>wheel_right_joint</right_wheel_joint_name>
-        <wheel_separation>0.235</wheel_separation>
-        <wheel_diameter>0.070</wheel_diameter>
-        <torque>1.0</torque>
-        <velocity_command_timeout>0.6</velocity_command_timeout>
-        <cliff_sensor_left_name>cliff_sensor_left</cliff_sensor_left_name>
-        <cliff_sensor_right_name>cliff_sensor_right</cliff_sensor_right_name>
-        <cliff_detection_threshold>0.04</cliff_detection_threshold>
-        <bumper_name>bumpers</bumper_name>
-        <imu_name>imu</imu_name>
+      <plugin name="gazebo_ros_imu_controller" filename="libgazebo_ros_imu.so">
+        <topicName>/neato/imu</topicName>
+        <bodyName>imu_link</bodyName>
       </plugin>
     </gazebo>
+    <gazebo>
+      <plugin name="differential_drive_controller" filename="libgazebo_ros_diff_drive.so">
+      <alwaysOn>true</alwaysOn>
+      <updateRate>10</updateRate>
+      <leftJoint>wheel_left_joint</leftJoint>
+      <rightJoint>wheel_right_joint</rightJoint>
+      <wheelSeparation>0.235</wheelSeparation>
+      <wheelDiameter>0.070</wheelDiameter>
+      <torque>1.0</torque>
+      <commandTopic>/neato/cmd_vel</commandTopic>
+      <odometryTopic>/neato/odom</odometryTopic>
+      <odometryFrame>base_link</odometryFrame>
+      <robotBaseFrame>base_footprint</robotBaseFrame>
+    </plugin>
+  </gazebo>
   </xacro:macro>
 </robot>

Commit message: Fixed bugs in robot description. SLAM navigation is now working.

File: neato_description/urdf/neato.urdf.xacro (robot description, xacro)
@@ -48,6 +48,6 @@
       <parent link="base_link"/>
       <child link="wheel_left_link"/>
-      <origin xyz="0.00 ${0.235/2} 0.0250" rpy="${M_PI/2} 0 ${M_PI}"/>
-      <axis xyz="0 0 1"/>
+      <origin xyz="0.00 ${0.235/2} 0.0250" rpy="0 0 0"/>
+      <axis xyz="0 1 0"/>
     </joint>
     <link name="wheel_left_link">
@@ -56,11 +56,11 @@
           <mesh filename="package://neato_description/meshes/wheel.dae"/>
         </geometry>
-        <origin xyz="0 0 0" rpy="0 0 0"/>
+        <origin xyz="0 0 0" rpy="${M_PI/2} 0 0"/>
       </visual>
       <collision>
         <geometry>
-          <cylinder length="0.0206" radius="0.0352"/>
-        </geometry>
-        <origin rpy="0 0 0" xyz="0 0 0"/>
+          <cylinder length="0.0206" radius="0.035"/>
+        </geometry>
+        <origin xyz="0 0 0" rpy="${M_PI/2} 0 0"/>
       </collision>
       <inertial>
@@ -75,6 +75,6 @@
       <parent link="base_link"/>
       <child link="wheel_right_link"/>
-      <origin xyz="0.00 -${0.235/2} 0.0250" rpy="${M_PI/2} 0 ${M_PI}"/>
-      <axis xyz="0 0 1"/>
+      <origin xyz="0.00 -${0.235/2} 0.0250" rpy="0 0 0"/>
+      <axis xyz="0 1 0"/>
     </joint>
     <link name="wheel_right_link">
@@ -83,11 +83,11 @@
           <mesh filename="package://neato_description/meshes/wheel.dae"/>
         </geometry>
-        <origin xyz="0 0 0" rpy="0 0 0"/>
+        <origin xyz="0 0 0" rpy="${M_PI/2} 0 0"/>
       </visual>
       <collision>
         <geometry>
-          <cylinder length="0.0206" radius="0.0350"/>
-        </geometry>
-        <origin rpy="0 0 0" xyz="0 0 0"/>
+          <cylinder length="0.0206" radius="0.035"/>
+        </geometry>
+        <origin xyz="0 0 0" rpy="${M_PI/2} 0 0"/>
       </collision>
       <inertial>
@@ -109,5 +109,5 @@
           <cylinder length="0.0176" radius="0.01"/>
         </geometry>
-        <origin rpy="0 0 0" xyz="0 0 0"/>
+        <origin xyz="0 0 0" rpy="0 0 0"/>
       </collision>
       <inertial>
@@ -129,5 +129,5 @@
           <cylinder length="0.0176" radius="0.01"/>
         </geometry>
-        <origin rpy="0 0 0" xyz="0 0 0"/>
+        <origin xyz="0 0 0" rpy="0 0 0"/>
       </collision>
       <inertial>
@@ -149,5 +149,5 @@
           <cylinder length="0.0176" radius="0.01"/>
         </geometry>
-        <origin rpy="0 0 0" xyz="0 0 0"/>
+        <origin xyz="0 0 0" rpy="0 0 0"/>
       </collision>
       <inertial>
@@ -169,5 +169,5 @@
           <cylinder length="0.0176" radius="0.01"/>
         </geometry>
-        <origin rpy="0 0 0" xyz="0 0 0"/>
+        <origin xyz="0 0 0" rpy="0 0 0"/>
       </collision>
       <inertial>

File: neato_description/urdf/neato_gazebo.urdf.xacro (robot description, xacro)
@@ -181,6 +181,6 @@
       <alwaysOn>true</alwaysOn>
       <updateRate>10</updateRate>
-      <leftJoint>wheel_left_joint</leftJoint>
-      <rightJoint>wheel_right_joint</rightJoint>
+      <leftJoint>wheel_right_joint</leftJoint>
+      <rightJoint>wheel_left_joint</rightJoint>
       <wheelSeparation>0.235</wheelSeparation>
       <wheelDiameter>0.070</wheelDiameter>

Commit message: Provide launchfile for just the description

File: neato_description/urdf/neato.urdf.xacro (robot description, xacro)
@@ -11,10 +11,4 @@
   <!-- neato -->
   <xacro:macro name="neato">
-    <link name="base_footprint"/>
-    <joint name="base_joint" type="fixed">
-      <origin xyz="0 0 0" rpy="0 0 0" />
-      <parent link="base_footprint"/>
-      <child link="base_link" />
-    </joint>
     <link name="base_link">
       <visual>
@@ -45,4 +39,10 @@
       </inertial>
     </link>
+    <joint name="base_footprint_joint" type="fixed">
+      <origin xyz="0 0 0" rpy="0 0 0" />
+      <parent link="base_link"/>
+      <child link="base_footprint" />
+    </joint>
+    <link name="base_footprint"/>
     <joint name="wheel_left_joint" type="continuous">
       <parent link="base_link"/>
