Commit message: Spawning gazebo neato entity

File: neato_description/urdf/neato.urdf.xacro (robot description, xacro)
@@ -6,9 +6,15 @@
       neato_description/launch/view_model.launch
  -->
-<robot name="neato" xmlns:xacro="http://ros.org/wiki/xacro">
+<robot name="neato" xmlns:xacro="http://www.ros.org/wiki/xacro">
   <xacro:include filename="$(find neato_description)/urdf/common_properties.urdf.xacro"/>
   <xacro:include filename="$(find neato_description)/urdf/neato_gazebo.urdf.xacro"/>
   <!-- neato -->
   <xacro:macro name="neato">
+    <link name="base_footprint"/>
+    <joint name="base_joint" type="fixed">
+      <origin xyz="0 0 0" rpy="0 0 0" />
+      <parent link="base_footprint"/>
+      <child link="base_link" />
+    </joint>
     <link name="base_link">
       <visual>
@@ -39,10 +45,4 @@
       </inertial>
     </link>
-    <joint name="base_footprint_joint" type="fixed">
-      <origin xyz="0 0 0" rpy="0 0 0" />
-      <parent link="base_link"/>
-      <child link="base_footprint" />
-    </joint>
-    <link name="base_footprint"/>
     <joint name="wheel_left_joint" type="continuous">
       <parent link="base_link"/>

File: neato_description/urdf/neato_gazebo.urdf.xacro (robot description, xacro)
@@ -69,6 +69,7 @@
       </sensor>
     </gazebo>
+    <!--
     <gazebo reference="cliff_sensor_left_link">
-      <sensor type="gpu_ray" name="cliff_sensor_left">
+      <sensor type="ray_sensor" name="cliff_sensor_left">
         <always_on>true</always_on>
         <update_rate>50</update_rate>
@@ -95,13 +96,21 @@
       </sensor>
     </gazebo>
+    -->
+    <!--
     <gazebo reference="cliff_sensor_right_link">
-      <sensor type="gpu_ray" name="cliff_sensor_right">
-        <always_on>true</always_on>
-        <update_rate>50</update_rate>
+      <plugin name="gazebo_ros_laser_controller" filename="libgazebo_ros_ray_sensor.so">
+          <ros>
+            <argument>~/out:=cliff_right</argument>
+          </ros>
+          <frame_name>laser_link</frame_name>
+      </plugin>
+      <sensor type="ray" name="cliff_sensor_right">
+        <always_on>true</always_on>
+        <update_rate>5</update_rate>
         <visualize>true</visualize>
         <ray>
           <scan>
             <horizontal>
-              <samples>50</samples>
+              <samples>1</samples>
               <resolution>1.0</resolution>
               <min_angle>-0.0436</min_angle>
@@ -115,14 +124,18 @@
           </range>
         </ray>
-        <plugin name="gazebo_ros_laser_controller" filename="libgazebo_ros_gpu_laser.so">
-          <topicName>/neato/cliff_right</topicName>
-          <frameName>cliff_sensor_right_link</frameName>
-        </plugin>
-      </sensor>
-    </gazebo>
+      </sensor>
+    </gazebo>
+    -->
     <gazebo reference="laser_link">
-      <sensor type="gpu_ray" name="laser">
-        <always_on>true</always_on>
-        <update_rate>50</update_rate>
+      <sensor type="ray" name="laser">
+        <plugin name="gazebo_ros_laser_controller" filename="libgazebo_ros_ray_sensor.so">
+          <ros>
+            <argument>~/out:=scan</argument>
+          </ros>
+          <output_type>sensor_msgs/LaserScan</output_type>
+          <frame_name>laser_link</frame_name>
+        </plugin>
+        <always_on>true</always_on>
+        <update_rate>5</update_rate>
         <visualize>true</visualize>
         <ray>
@@ -141,14 +154,18 @@
           </range>
         </ray>
-        <plugin name="gazebo_ros_laser_controller" filename="libgazebo_ros_gpu_laser.so">
-          <topicName>/neato/laser</topicName>
-          <frameName>laser_link</frameName>
-        </plugin>
       </sensor>
     </gazebo>
     <gazebo reference="imu_link">
-      <sensor type="imu" name="imu">
-        <always_on>true</always_on>
-        <update_rate>50</update_rate>
+      <sensor type="imu" name="neato_imu">
+        <plugin name="gazebo_ros_imu_controller" filename="libgazebo_ros_imu_sensor.so">
+          <ros>
+            <argument>~/out:=imu</argument>
+          </ros>
+          <output_type>sensor_msgs/msg/Imu</output_type>
+          <body_name>imu_link</body_name>
+          <frame_name>imu_link</frame_name>
+        </plugin>
+        <always_on>true</always_on>
+        <update_rate>10</update_rate>
         <visualize>false</visualize>
         <imu>
@@ -172,24 +189,17 @@
     </gazebo>
     <gazebo>
-      <plugin name="gazebo_ros_imu_controller" filename="libgazebo_ros_imu.so">
-        <topicName>/neato/imu</topicName>
-        <bodyName>imu_link</bodyName>
+      <plugin name="differential_drive_controller" filename="libgazebo_ros_diff_drive.so">
+        <update_rate>10</update_rate>
+        <left_joint>wheel_right_joint</left_joint>
+        <right_joint>wheel_left_joint</right_joint>
+        <wheel_separation>0.235</wheel_separation>
+        <wheel_diameter>0.070</wheel_diameter>
+        <torque>1.0</torque>
+        <command_topic>cmd_vel</command_topic>
+        <odometry_topic>odom</odometry_topic>
+        <odometry_frame>odom</odometry_frame>
+        <robot_base_frame>base_footprint</robot_base_frame>
       </plugin>
     </gazebo>
-    <gazebo>
-      <plugin name="differential_drive_controller" filename="libgazebo_ros_diff_drive.so">
-      <alwaysOn>true</alwaysOn>
-      <updateRate>10</updateRate>
-      <leftJoint>wheel_right_joint</leftJoint>
-      <rightJoint>wheel_left_joint</rightJoint>
-      <wheelSeparation>0.235</wheelSeparation>
-      <wheelDiameter>0.070</wheelDiameter>
-      <torque>1.0</torque>
-      <commandTopic>cmd_vel</commandTopic>
-      <odometryTopic>odom</odometryTopic>
-      <odometryFrame>odom</odometryFrame>
-      <robotBaseFrame>base_footprint</robotBaseFrame>
-    </plugin>
-  </gazebo>
   </xacro:macro>
 </robot>

Commit message: Fix links and publish odom from gazebo

File: neato_description/urdf/neato.urdf.xacro (robot description, xacro)
@@ -11,10 +11,4 @@
   <!-- neato -->
   <xacro:macro name="neato">
-    <link name="base_footprint"/>
-    <joint name="base_joint" type="fixed">
-      <origin xyz="0 0 0" rpy="0 0 0" />
-      <parent link="base_footprint"/>
-      <child link="base_link" />
-    </joint>
     <link name="base_link">
       <visual>
@@ -45,4 +39,10 @@
       </inertial>
     </link>
+    <link name="base_footprint"/>
+    <joint name="base_joint" type="fixed">
+      <origin xyz="0 0 0" rpy="0 0 0" />
+      <parent link="base_link"/>
+      <child link="base_footprint" />
+    </joint>
     <joint name="wheel_left_joint" type="continuous">
       <parent link="base_link"/>

File: neato_description/urdf/neato_gazebo.urdf.xacro (robot description, xacro)
@@ -195,9 +195,14 @@
         <wheel_separation>0.235</wheel_separation>
         <wheel_diameter>0.070</wheel_diameter>
-        <torque>1.0</torque>
+        <max_wheel_torque>20</max_wheel_torque>
+        <max_wheel_acceleration>1.0</max_wheel_acceleration>
         <command_topic>cmd_vel</command_topic>
+        <!-- output -->
+        <publish_odom>true</publish_odom>
+        <publish_odom_tf>true</publish_odom_tf>
+        <!-- <publish_wheel_tf>true</publish_wheel_tf> -->
         <odometry_topic>odom</odometry_topic>
         <odometry_frame>odom</odometry_frame>
-        <robot_base_frame>base_footprint</robot_base_frame>
+        <robot_base_frame>base_link</robot_base_frame>
       </plugin>
     </gazebo>

Commit message: Cleaned up models and launchfiles produces decent result running slam in simulation

File: neato_description/urdf/neato.urdf.xacro (robot description, xacro)
@@ -21,5 +21,5 @@
       <collision>
         <geometry>
-          <cylinder length="0.06" radius="0.15"/>
+          <cylinder length="0.04" radius="0.15"/>
         </geometry>
         <origin xyz="-0.01 0 0.03" rpy="0 0 0"/>
@@ -27,5 +27,5 @@
       <collision>
         <geometry>
-          <box size="0.16 0.3 0.06"/>
+          <box size="0.16 0.3 0.05"/>
         </geometry>
         <origin xyz="0.08 0 0.03" rpy="0 0 0"/>
@@ -224,5 +224,5 @@
     </link>
     <joint name="laser_joint" type="fixed">
-      <origin xyz="-0.084 0 0.066" rpy="0 0 0" />
+      <origin xyz="-0.084 0 0.1" rpy="0 0 0" />
       <parent link="base_link"/>
       <child link="laser_link" />

File: neato_description/urdf/neato_gazebo.urdf.xacro (robot description, xacro)
@@ -149,8 +149,13 @@
           </scan>
           <range>
-            <min>0.1</min>
+            <min>0.3</min>
             <max>5</max>
             <resolution>1</resolution>
           </range>
+          <noise>
+            <type>gaussian</type>
+            <mean>0.0</mean>
+            <stddev>0.0</stddev>
+          </noise>
         </ray>
       </sensor>

Commit message: Publishes bumper states about single bumper
Signed-off-by: Emerson Knapp <eknapp@amazon.com>

File: neato_description/urdf/neato.urdf.xacro (robot description, xacro)
@@ -19,5 +19,5 @@
         <material name="dark_grey"/>
       </visual>
-      <collision>
+      <collision name="body">
         <geometry>
           <cylinder length="0.04" radius="0.15"/>
@@ -25,10 +25,30 @@
         <origin xyz="-0.01 0 0.03" rpy="0 0 0"/>
       </collision>
-      <collision>
-        <geometry>
-          <box size="0.16 0.3 0.05"/>
-        </geometry>
-        <origin xyz="0.08 0 0.03" rpy="0 0 0"/>
-      </collision>
+      <collision name="left_bumper">
+        <geometry>
+          <box size="0.16 0.3 0.05"/>
+        </geometry>
+        <origin xyz="0.08 0 0.03" rpy="0 0 0"/>
+      </collision>
+      <!--
+      <collision name="left_front_bumper">
+        <geometry>
+          <box size="0.16 0.3 0.05"/>
+        </geometry>
+        <origin xyz="0.08 0 0.03" rpy="0 0 0"/>
+      </collision>
+      <collision name="">
+        <geometry>
+          <box size="0.16 0.3 0.05"/>
+        </geometry>
+        <origin xyz="0.08 0 0.03" rpy="0 0 0"/>
+      </collision>
+      <collision name="bumper">
+        <geometry>
+          <box size="0.16 0.3 0.05"/>
+        </geometry>
+        <origin xyz="0.08 0 0.03" rpy="0 0 0"/>
+      </collision>
+      -->
       <inertial>
         <origin xyz="0.01 0 0"/>

File: neato_description/urdf/neato_gazebo.urdf.xacro (robot description, xacro)
@@ -56,10 +56,10 @@
       <mu1>0.3</mu1>
       <mu2>0.3</mu2>
-      <sensor type="contact" name="bumpers">
+      <sensor type="contact" name="left_bumper">
         <always_on>1</always_on>
         <update_rate>50.0</update_rate>
         <visualize>true</visualize>
         <contact>
-          <collision>base_footprint_collision_base_link</collision>
+          <collision>base_link_fixed_joint_lump__left_bumper_collision_1</collision>
         </contact>
         <plugin name="gazebo_ros_bumper_controller" filename="libgazebo_ros_bumper.so">
@@ -68,4 +68,12 @@
         </plugin>
       </sensor>
+      <!--
+      <sensor type="contact" name="left_front_bumper">
+      </sensor>
+      <sensor type="contact" name="right_front_bumper">
+      </sensor>
+      <sensor type="contact" name="right_bumper">
+      </sensor>
+      -->
     </gazebo>
     <!--

Commit message: Collision shape/size of all 4 bumpers
Signed-off-by: Emerson Knapp <eknapp@amazon.com>

File: neato_description/urdf/neato.urdf.xacro (robot description, xacro)
@@ -27,28 +27,26 @@
       <collision name="left_bumper">
         <geometry>
-          <box size="0.16 0.3 0.05"/>
-        </geometry>
-        <origin xyz="0.08 0 0.03" rpy="0 0 0"/>
-      </collision>
-      <!--
-      <collision name="left_front_bumper">
-        <geometry>
-          <box size="0.16 0.3 0.05"/>
-        </geometry>
-        <origin xyz="0.08 0 0.03" rpy="0 0 0"/>
-      </collision>
-      <collision name="">
-        <geometry>
-          <box size="0.16 0.3 0.05"/>
-        </geometry>
-        <origin xyz="0.08 0 0.03" rpy="0 0 0"/>
-      </collision>
-      <collision name="bumper">
-        <geometry>
-          <box size="0.16 0.3 0.05"/>
-        </geometry>
-        <origin xyz="0.08 0 0.03" rpy="0 0 0"/>
-      </collision>
-      -->
+          <box size="0.15 0.05 0.05"/>
+        </geometry>
+        <origin xyz="0.07 0.125 0.03" rpy="0 0 0"/>
+      </collision>
+      <collision name="right_bumper">
+        <geometry>
+          <box size="0.15 0.05 0.05"/>
+        </geometry>
+        <origin xyz="0.07 -0.125 0.03" rpy="0 0 0"/>
+      </collision>
+      <collision name="front_right_bumper">
+        <geometry>
+          <box size="0.05 0.13 0.05"/>
+        </geometry>
+        <origin xyz="0.135 -0.07 0.03" rpy="0 0 0"/>
+      </collision>
+      <collision name="front_left_bumper">
+        <geometry>
+          <box size="0.05 0.13 0.05"/>
+        </geometry>
+        <origin xyz="0.135 0.07 0.03" rpy="0 0 0"/>
+      </collision>
       <inertial>
         <origin xyz="0.01 0 0"/>

Commit message: Add TODO note about how to silence KDL warning
Signed-off-by: Emerson Knapp <eknapp@amazon.com>

File: neato_description/urdf/neato.urdf.xacro (robot description, xacro)
@@ -11,4 +11,7 @@
   <!-- neato -->
   <xacro:macro name="neato">
+    <!-- TODO(emersonknapp) KDL complains about inertia in root link, but adding a dummy changes
+    the names of the collision lumps for the contact sensors. Use new link frames for bumpers
+    instead of collisions on the base_link -->
     <link name="base_link">
       <visual>
@@ -57,10 +60,4 @@
       </inertial>
     </link>
-    <link name="base_footprint"/>
-    <joint name="base_joint" type="fixed">
-      <origin xyz="0 0 0" rpy="0 0 0" />
-      <parent link="base_link"/>
-      <child link="base_footprint" />
-    </joint>
     <joint name="wheel_left_joint" type="continuous">
       <parent link="base_link"/>
