Commit message: Neato diff_drive Load implementation
Signed-off-by: Emerson Knapp <emerson.b.knapp@gmail.com>

File: neato_description/urdf/neato_gazebo.urdf.xacro (robot description, xacro)
@@ -3,5 +3,5 @@
   <xacro:macro name="neato_sim">
     <gazebo reference="base_link">
-      <material>Gazebo/DarkGrey</material>
+      <material>Gazebo/LightGrey</material>
     </gazebo>
     <gazebo reference="wheel_left_link">
@@ -193,4 +193,25 @@
       </sensor>
     </gazebo>
+    <!-- This version is for the NeatoWheelCommand controller. Commented out parameters, not sure if we need them yet. -->
+    <gazebo>
+      <plugin name="drive_controller" filename="libneato_gazebo_diff_drive.so">
+        <!-- <update_rate>10</update_rate> -->
+        <left_joint>wheel_left_joint</left_joint>
+        <right_joint>wheel_right_joint</right_joint>
+        <!-- <wheel_separation>0.235</wheel_separation> -->
+        <wheel_diameter>0.070</wheel_diameter>
+        <max_wheel_torque>20</max_wheel_torque>
+        <max_wheel_acceleration>1.0</max_wheel_acceleration>
+        <command_topic>neato_cmd</command_topic>
+        <publish_odom>true</publish_odom>
+        <publish_odom_tf>true</publish_odom_tf>
+        <publish_wheel_tf>true</publish_wheel_tf>
+        <odometry_topic>odom</odometry_topic>
+        <odometry_frame>odom</odometry_frame>
+        <robot_base_frame>base_link</robot_base_frame>
+      </plugin>
+    </gazebo>
+    <!-- This version is for the normal diff_drive controller that takes in Twist msgs -->
+    <!--
     <gazebo>
       <plugin name="differential_drive_controller" filename="libgazebo_ros_diff_drive.so">
@@ -203,5 +224,4 @@
         <max_wheel_acceleration>1.0</max_wheel_acceleration>
         <command_topic>cmd_vel</command_topic>
-        <!-- output -->
         <publish_odom>true</publish_odom>
         <publish_odom_tf>true</publish_odom_tf>
@@ -212,4 +232,5 @@
       </plugin>
     </gazebo>
+    -->
   </xacro:macro>
 </robot>

Commit message: Create a useful RViz, launch it, stop initial robot drift
Signed-off-by: Emerson Knapp <emerson.b.knapp@gmail.com>

File: neato_description/urdf/neato_gazebo.urdf.xacro (robot description, xacro)
@@ -3,5 +3,5 @@
   <xacro:macro name="neato_sim">
     <gazebo reference="base_link">
-      <material>Gazebo/LightGrey</material>
+      <material>Gazebo/DarkGrey</material>
     </gazebo>
     <gazebo reference="wheel_left_link">

Commit message: Connect four bumpers to bumper topics
Signed-off-by: Emerson Knapp <eknapp@amazon.com>

File: neato_description/urdf/neato_gazebo.urdf.xacro (robot description, xacro)
@@ -3,5 +3,5 @@
   <xacro:macro name="neato_sim">
     <gazebo reference="base_link">
-      <material>Gazebo/DarkGrey</material>
+      <material>Gazebo/White</material>
     </gazebo>
     <gazebo reference="wheel_left_link">
@@ -58,5 +58,5 @@
       <sensor type="contact" name="left_bumper">
         <always_on>1</always_on>
-        <update_rate>50.0</update_rate>
+        <update_rate>10.0</update_rate>
         <visualize>true</visualize>
         <contact>
@@ -64,16 +64,48 @@
         </contact>
         <plugin name="gazebo_ros_bumper_controller" filename="libgazebo_ros_bumper.so">
-          <bumperTopicName>/neato/bumper</bumperTopicName>
-          <frameName>world</frameName>
-        </plugin>
-      </sensor>
-      <!--
-      <sensor type="contact" name="left_front_bumper">
-      </sensor>
-      <sensor type="contact" name="right_front_bumper">
+          <ros>
+            <remapping>/bumper_states:=/bumper/left</remapping>
+          </ros>
+        </plugin>
       </sensor>
       <sensor type="contact" name="right_bumper">
-      </sensor>
-      -->
+        <always_on>1</always_on>
+        <update_rate>10.0</update_rate>
+        <visualize>true</visualize>
+        <contact>
+          <collision>base_link_fixed_joint_lump__right_bumper_collision_2</collision>
+        </contact>
+        <plugin name="gazebo_ros_bumper_controller" filename="libgazebo_ros_bumper.so">
+          <ros>
+            <remapping>/bumper_states:=/bumper/right</remapping>
+          </ros>
+        </plugin>
+      </sensor>
+      <sensor type="contact" name="front_left_bumper">
+        <always_on>1</always_on>
+        <update_rate>10.0</update_rate>
+        <visualize>true</visualize>
+        <contact>
+          <collision>base_link_fixed_joint_lump__front_left_bumper_collision_4</collision>
+        </contact>
+        <plugin name="gazebo_ros_bumper_controller" filename="libgazebo_ros_bumper.so">
+          <ros>
+            <remapping>/bumper_states:=/bumper/front_left</remapping>
+          </ros>
+        </plugin>
+      </sensor>
+      <sensor type="contact" name="front_right_bumper">
+        <always_on>1</always_on>
+        <update_rate>10.0</update_rate>
+        <visualize>true</visualize>
+        <contact>
+          <collision>base_link_fixed_joint_lump__front_right_bumper_collision_3</collision>
+        </contact>
+        <plugin name="gazebo_ros_bumper_controller" filename="libgazebo_ros_bumper.so">
+          <ros>
+            <remapping>/bumper_states:=/bumper/front_right</remapping>
+          </ros>
+        </plugin>
+      </sensor>
     </gazebo>
     <!--
@@ -139,5 +171,5 @@
         <plugin name="gazebo_ros_laser_controller" filename="libgazebo_ros_ray_sensor.so">
           <ros>
-            <argument>~/out:=scan</argument>
+            <remapping>~/out:=/scan</remapping>
           </ros>
           <output_type>sensor_msgs/LaserScan</output_type>
@@ -173,9 +205,10 @@
         <plugin name="gazebo_ros_imu_controller" filename="libgazebo_ros_imu_sensor.so">
           <ros>
-            <argument>~/out:=imu</argument>
+            <remapping>~/out:=/imu</remapping>
           </ros>
           <output_type>sensor_msgs/msg/Imu</output_type>
           <body_name>imu_link</body_name>
           <frame_name>imu_link</frame_name>
+          <initial_orientation_as_reference>false</initial_orientation_as_reference>
         </plugin>
         <always_on>true</always_on>
@@ -204,8 +237,6 @@
     <gazebo>
       <plugin name="drive_controller" filename="libneato_gazebo_diff_drive.so">
-        <!-- <update_rate>10</update_rate> -->
         <left_joint>wheel_left_joint</left_joint>
         <right_joint>wheel_right_joint</right_joint>
-        <!-- <wheel_separation>0.235</wheel_separation> -->
         <wheel_diameter>0.070</wheel_diameter>
         <max_wheel_torque>20</max_wheel_torque>
